Commit message: added gazebo conf

File: description/robot_core.xacro (robot description, xacro)
@@ -34,4 +34,7 @@
       </visual>
    </link>
+   <gazebo reference="chassis">
+    <material>Gazebo/White</material>
+   </gazebo>
    <!-- LEFT WHEEL LINK -->
     <joint name="left_wheel_joint" type="continuous">
@@ -58,4 +61,7 @@
         </xacro:inertial_cylinder>
     </link>
+    <gazebo reference="left_wheel">
+    <material>Gazebo/Blue</material>
+   </gazebo>
     <!-- RIGHT WHEEL LINK -->
     <joint name="right_wheel_joint" type="continuous">
@@ -81,4 +87,7 @@
         </xacro:inertial_cylinder>
     </link>
+    <gazebo reference="right_wheel">
+    <material>Gazebo/Blue</material>
+   </gazebo>
     <!-- CASTER WHEEL LINK -->
     <joint name="caster_wheel_joint" type="fixed">
@@ -103,3 +112,8 @@
         </xacro:inertial_sphere>
     </link>
+    <gazebo reference="caster_wheel">
+       <material>Gazebo/Black</material>
+       <mu1 value="0.001"/>
+       <mu2 value="0.001"/>
+    </gazebo>
 </robot>
